File: circuits/board/watts_meter.brd (EAGLE design)
At the start: 100.3 x 70 mm, 35 parts

Commit message: .
Parts:
- moved E$3 0.64 mm to (86.4, 21.0)
Changed lines of the file:
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@@
 <?xml version="1.0" encoding="utf-8"?>
 <!DOCTYPE eagle SYSTEM "eagle.dtd">
-<eagle version="9.6.2">
+<eagle version="8.5.2">
 <drawing>
 <settings>
@@
 <param name="checkStop" value="0"/>
 <param name="checkValues" value="0"/>
-<param name="checkNames" value="1"/>
-<param name="checkWireStubs" value="1"/>
-<param name="checkPolygonWidth" value="0"/>
 <param name="useDiameter" value="13"/>
 <param name="maxErrors" value="50"/>
@@
 <attribute name="VALUE" x="106.045" y="7.366" size="1.27" layer="27" ratio="10" rot="R270"/>
 </element>
-<element name="E$3" library="con-lstb" library_urn="urn:adsk.eagle:library:162" package="MA05-1" package3d_urn="urn:adsk.eagle:package:8332/1" value="" x="86.36" y="21.59" smashed="yes" rot="R270">
-<attribute name="NAME" x="88.011" y="27.94" size="1.27" layer="25" ratio="10" rot="R270"/>
-<attribute name="VALUE" x="83.439" y="24.13" size="1.27" layer="27" ratio="10" rot="R270"/>
+<element name="E$3" library="con-lstb" library_urn="urn:adsk.eagle:library:162" package="MA05-1" package3d_urn="urn:adsk.eagle:package:8332/1" value="" x="86.36" y="20.955" smashed="yes" rot="R270">
+<attribute name="NAME" x="88.011" y="27.305" size="1.27" layer="25" ratio="10" rot="R270"/>
+<attribute name="VALUE" x="83.439" y="23.495" size="1.27" layer="27" ratio="10" rot="R270"/>
 </element>
 <element name="E$6" library="led" library_urn="urn:adsk.eagle:library:259" package="LED3MM" package3d_urn="urn:adsk.eagle:package:15797/1" value="" x="107.95" y="64.135" smashed="yes">
@@
 <element name="E$5" library="eagle-ltspice" package="0204/7" value="10k" x="45.72" y="17.145" smashed="yes">
 <attribute name="NAME" x="43.18" y="18.4404" size="0.9906" layer="25" ratio="10"/>
-<attribute name="VALUE" x="44.0944" y="15.3924" size="0.9906" layer="27" ratio="10"/>
+<attribute name="VALUE" x="44.0944" y="14.7574" size="0.9906" layer="27" ratio="10"/>
 </element>
 <element name="E$16" library="rcl" library_urn="urn:adsk.eagle:library:334" package="C025-024X044" package3d_urn="urn:adsk.eagle:package:23630/1" value="" x="41.91" y="22.86" smashed="yes" rot="R90">
@@
 <wire x1="59.69" y1="17.78" x2="63.5" y2="22.86" width="0" layer="19" extent="1-1"/>
 <wire x1="76.2" y1="18.415" x2="63.5" y2="22.86" width="0" layer="19" extent="1-1"/>
-<wire x1="86.36" y1="19.05" x2="76.2" y2="18.415" width="0" layer="19" extent="1-1"/>
-<wire x1="86.36" y1="21.59" x2="86.36" y2="19.05" width="0" layer="19" extent="1-1"/>
-<wire x1="86.36" y1="24.13" x2="86.36" y2="21.59" width="0" layer="19" extent="1-1"/>
-<wire x1="86.36" y1="26.67" x2="86.36" y2="24.13" width="0" layer="19" extent="1-1"/>
-<wire x1="86.36" y1="16.51" x2="86.36" y2="19.05" width="0" layer="19" extent="1-1"/>
+<wire x1="86.36" y1="18.415" x2="76.2" y2="18.415" width="0" layer="19" extent="1-1"/>
+<wire x1="86.36" y1="20.955" x2="86.36" y2="18.415" width="0" layer="19" extent="1-1"/>
+<wire x1="86.36" y1="23.495" x2="86.36" y2="20.955" width="0" layer="19" extent="1-1"/>
+<wire x1="86.36" y1="26.035" x2="86.36" y2="23.495" width="0" layer="19" extent="1-1"/>
+<wire x1="86.36" y1="15.875" x2="86.36" y2="18.415" width="0" layer="19" extent="1-1"/>
 <wire x1="50.165" y1="39.37" x2="60.96" y2="30.48" width="0" layer="19" extent="1-1"/>
 <wire x1="39.37" y1="37.56" x2="50.165" y2="39.37" width="0" layer="19" extent="1-1"/>
@@
 </signal>
 </signals>
-<mfgpreviewcolors>
-<mfgpreviewcolor name="soldermaskcolor" color="0xC8008000"/>
-<mfgpreviewcolor name="silkscreencolor" color="0xFFFEFEFE"/>
-<mfgpreviewcolor name="backgroundcolor" color="0xFF282828"/>
-<mfgpreviewcolor name="coppercolor" color="0xFFFFBF00"/>
-<mfgpreviewcolor name="substratecolor" color="0xFF786E46"/>
-</mfgpreviewcolors>
 </board>
 </drawing>

Commit message: .
Parts:
- removed E$21: 10k, eagle-ltspice:0204/7
- added E$22: 103, rcl:RTRIM3296W
- E$17: value 4.3K 3W -> 2.2K
- E$20: value 2k -> 103; device eagle-ltspice:0204/7 -> rcl:RTRIM3296W
- moved E$44 13.1 mm to (74.9, 54.0), turned to 180 degrees
- moved PROGRAM 8.84 mm to (87.6, 56.5)
- moved E$33 8.03 mm to (70.5, 54.0)
- moved E$5 6.35 mm to (45.7, 10.8)
- moved E$10 5.12 mm to (68.6, 11.4)
- moved E$3 4.62 mm to (85.1, 16.5)
- moved E$12 4.49 mm to (60.3, 12.1)
- moved E$15 4.45 mm to (76.2, 12.7)
- moved E$1 3.24 mm to (62.9, 23.5)
- moved E$20 2.94 mm to (71.7, 40.4), turned to 90 degrees
- moved E$34 1.42 mm to (48.9, 33.0)
- moved E$7 0.90 mm to (55.9, 38.7), turned to 180 degrees
Connections:
- removed net S$15: E$1.23, E$20.1, E$21.2, E$44.TP
- new net S$4: E$1.23, E$20.1, E$22.1, E$44.TP
- net GND: now also E$7.A; no longer E$7.C
- net S$8: now also E$22.2, E$7.C; no longer E$21.1, E$7.A
Other:
- board text added: "+"
- board text added: "-"

Commit message: .
Parts:
- added E$21, E$27: 10k, eagle-ltspice:0204/7
- moved PROGRAM 14.7 mm to (88.9, 41.9), turned to 90 degrees
- moved E$29 7.01 mm to (15.6, 62.2)
- moved E$8 5.85 mm to (38.1, 54.0)
- moved E$4 5.24 mm to (36.8, 39.4)
- moved E$34 5.12 mm to (43.8, 33.7)
- moved E$7 4.96 mm to (52.1, 41.9)
- moved E$5 4.62 mm to (47.0, 15.2)
- moved E$2 4.44 mm to (21.0, 41.9)
- moved E$20 3.81 mm to (71.7, 36.6)
- moved E$16 3.18 mm to (41.9, 19.7), turned to 180 degrees
- moved E$13 2.54 mm to (59.4, 58.4)
- moved E$33 2.01 mm to (71.1, 52.1)
- moved E$44 2.01 mm to (74.3, 52.1)
- moved E$22 1.91 mm to (71.7, 44.9)
- moved E$3 0.64 mm to (85.1, 15.9)
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Connections:
- net GND: now also E$21.2, E$27.1
- net S$16: now also E$21.1
- net S$4: now also E$27.2
Other:
- board text removed: "P"

Commit message: .
Parts:
- removed E$33, E$34, E$44: (no value), testpad:P1-17Y
- added E$32: (no value), con-lstb:MA03-1
- added E$36: (no value), Rembrandt Electronics - JST XH Connectors v1-0:JST-XH-04-PACKAGE-LONG-PAD
- added E$37: 5v1 zener, diodes-zener:DO35-7
- E$17: value 2.2K -> (none)
- E$20: value 103 -> 1.7k -103
- E$22: value 103 -> 8.2k - 103
- E$25: value 20k 0.5W -> 2.2k
- moved E$25 41.5 mm to (81.3, 26.0), turned to 180 degrees
- moved PROGRAM 35.4 mm to (83.2, 6.99), turned to 0 degrees
- moved E$29 35.4 mm to (5.71, 28.3), turned to 270 degrees
- moved E$3 35.2 mm to (52.1, 3.81), turned to 180 degrees
- moved E$2 31.9 mm to (30.5, 11.4), turned to 90 degrees
- moved E$17 30.2 mm to (86.3, 64.0), turned to 180 degrees
- moved E$7 29.2 mm to (70.5, 64.5), turned to 0 degrees
- moved E$24 25.4 mm to (5.71, 6.35), turned to 270 degrees
- moved E$5 23.9 mm to (24.1, 22.2), turned to 180 degrees
- moved E$4 19.1 mm to (48.3, 54.6), turned to 90 degrees
- moved E$20 18.5 mm to (88.8, 43.6)
- moved E$10 18.2 mm to (54.0, 22.2)
- moved E$22 17.9 mm to (88.8, 49.9)
- moved E$15 17.8 mm to (61.6, 22.2)
- moved E$12 17.7 mm to (46.4, 22.2)
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Connections:
- removed net GND: E$1.22, E$1.8, E$12.2, E$13.1, E$15.1, E$19.1, E$2.P$7, E$20.2, E$21.2, E$24.1, E$27.1, E$29.1, E$3.1, E$3.2, E$3.3, E$3.4, E$3.5, E$4.2, E$7.A, E$8.2
- removed net S$8: E$17.2, E$22.2, E$33.TP, E$7.C
- new net S$15: E$1.28, E$36.3
- new net S$18: E$19.1, E$24.1, E$29.1, E$32.2, E$36.1, E$4.2, E$8.2
- new net S$20: E$25.1, E$37.A
- new net S$21: E$17.2, E$22.2, E$7.A
- net 5V: now also E$1.22, E$1.8, E$12.2, E$13.1, E$15.1, E$17.1, E$2.P$7, E$20.2, E$21.1, E$25.2, E$27.2, E$3.1, E$3.2, E$3.3, E$3.4, E$3.5, E$32.1, E$36.2
- net S$16: now also E$20.1, E$22.1, E$27.1, E$37.C; no longer E$21.1, E$34.TP, E$8.3
- net S$4: now also E$21.2, E$8.3; no longer E$20.1, E$22.1, E$27.2, E$44.TP
- net S$9: now also E$7.C; no longer E$17.1
Other:
- board text removed: "G"
- board text removed: "S"

Commit message: .
Parts:
- added E$33: 220, eagle-ltspice:0204/7
- added E$34, E$39: 1uF, rcl:C025-024X044
- added E$38: 0.1uF, rcl:C025-024X044
- E$17: value (none) -> 2.2k
- E$20: value 1.7k -103 -> 2.2k; device rcl:RTRIM3296W -> eagle-ltspice:0204/7
- E$22: value 8.2k - 103 -> 2k - 202
- E$25: value 2.2k -> 5v1 zener; device eagle-ltspice:0204/7 -> diodes-zener:DO35-7
- E$36: value (none) -> display
- moved E$25 34.8 mm to (62.0, 55.0), turned to 0 degrees
- moved E$37 23.2 mm to (82.0, 52.0), turned to 180 degrees
- moved E$5 23.0 mm to (47.1, 23.2)
- moved E$20 22.5 mm to (82.0, 65.0), turned to 180 degrees
- moved E$1 18.1 mm to (66.3, 33.8)
- moved E$16 18.1 mm to (45.9, 28.7)
- moved E$12 18.0 mm to (64.4, 21.2)
- moved E$15 18.0 mm to (79.6, 21.2)
- moved E$10 18.0 mm to (72.0, 21.2)
- moved E$27 14.7 mm to (71.8, 55.0), turned to 180 degrees
- moved E$22 11.3 mm to (91.0, 61.0), turned to 180 degrees
- moved E$21 10.3 mm to (71.9, 52.0)
- moved E$17 10.00 mm to (82.0, 55.0)
- moved E$3 7.00 mm to (59.1, 3.81)
- moved E$36 6.40 mm to (24.3, 30.6)
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Connections:
- removed net S$18: E$19.1, E$24.1, E$29.1, E$32.2, E$36.1, E$4.2, E$8.2
- new net S$17: E$20.1, E$22.1
- new net S$19: E$1.24, E$17.1, E$22.2, E$27.1, E$37.C
- new net S$22: E$13.1, E$17.2, E$21.1, E$22.3, E$25.A, E$27.2, E$32.2, E$33.1, E$37.A, E$4.2, E$8.2
- new net S$8: E$20.2, E$7.A
- net 5V: now also E$1.21, E$25.C, E$29.1, E$33.2, E$36.1, E$38.2; no longer E$1.20, E$1.22, E$1.7, E$1.8, E$12.2, E$13.1, E$15.1, E$17.1, E$2.P$7, E$20.2, E$21.1, E$25.2, E$27.2, E$29.2, E$3.1, E$3.2, E$3.3, E$3.4, E$3.5, E$36.2, E$5.2
- net S$10: now also E$1.17; no longer E$1.16
- net S$11: now also E$1.18; no longer E$1.17
- net S$12: now also E$1.19; no longer E$1.18
- net S$16: now also E$1.27, E$36.4; no longer E$1.24, E$20.1, E$22.1, E$27.1, E$37.C
- net S$20: now also E$1.22, E$1.8, E$12.2, E$15.1, E$19.1, E$2.P$7, E$24.1, E$29.2, E$3.1, E$3.2, E$3.3, E$3.4, E$3.5, E$34.2, E$36.2, E$38.1, E$39.2, E$5.2, PROGRAM.P$6; no longer E$25.1, E$37.A
- net S$21: now also E$1.20, E$1.7, E$34.1, E$39.1; no longer E$17.2, E$22.2, E$7.A

Commit message: .
Parts:
- removed E$14: (no value), rcl:C025-024X044
- removed E$18: (no value), transistor-fet:TO92-
- removed E$23: (no value), ref-packages-longpad:E5-8,5
- removed E$26, E$35: (no value), con-lstb:MA04-1
- removed E$28: (no value), con-lstb:MA06-1
- removed E$30: (no value), discrete:RS-2,5
- removed E$31: (no value), pinhead:2X02/90
- removed E$45: (no value), 74xx-us:DIL08
- added E$41, E$42, E$43, E$46, E$47, E$48, E$49, E$50, E$51, E$52, E$53, E$54, E$56, E$57, E$58, E$59, E$60, E$61, E$62, E$63, E$64, E$65, E$66, E$67, E$68, E$69, E$70, E$71, E$72, E$73, E$74, E$75, E$76, E$77: (no value), solpad:LSP10
- added E$44: tx_to_multiplx, testpad:P1-17Y
- E$11: device rcl:C025-024X044 -> solpad:LSP10
- E$17: value 2.2k -> (none); device eagle-ltspice:0204/7 -> switch:TL1105
- E$24: value 5V -> 123; device con-wago-508:W237-132 -> testpad:P1-17Y
- E$3: value (none) -> ground-group
- E$6: device led:LED3MM -> solpad:LSP10
- E$8: value ACS758LCB 50U -> 123; device ACS758LCB-100B-PFF-T:XDCR_ACS770KCB-150U-PFF-T -> testpad:P1-17Y
- E$9: value (none) -> 123; device rcl:C025-024X044 -> testpad:P1-17Y
- moved E$8 72.4 mm to (94.5, 52.7), turned to 180 degrees
- moved E$24 69.2 mm to (58.2, 51.5), turned to 90 degrees
- moved E$17 68.8 mm to (20.2, 24.7)
- moved E$9 38.4 mm to (77.9, 56.8), turned to 90 degrees
- moved E$11 26.9 mm to (90.0, 50.4), turned to 0 degrees
- moved E$27 20.4 mm to (55.0, 43.6), turned to 90 degrees
- moved E$6 19.9 mm to (90.0, 55.5)
- moved E$21 16.4 mm to (57.6, 43.8), turned to 270 degrees
- moved E$22 8.06 mm to (90.0, 53.0)
- moved PROGRAM 8.00 mm to (91.2, 6.99)
- moved E$4 7.07 mm to (48.3, 47.6)
- moved E$32 7.00 mm to (44.5, 48.9)
- moved E$25 6.25 mm to (68.2, 54.2)
- moved E$36 5.36 mm to (24.0, 35.9)
- moved E$29 5.10 mm to (10.7, 29.3)
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Connections:
- removed net S$22: E$13.1, E$17.2, E$21.1, E$22.3, E$25.A, E$27.2, E$32.2, E$33.1, E$37.A, E$4.2, E$8.2
- removed net S$4: E$1.23, E$21.2, E$8.3
- new net S$18: E$1.22, E$1.8, E$12.2, E$13.1, E$15.1, E$17.4, E$19.1, E$2.P$7, E$21.1, E$22.3, E$25.A, E$27.2, E$29.2, E$3.1, E$3.2, E$3.3, E$3.4, E$3.5, E$32.2, E$34.2, E$36.2, E$37.A, E$38.1, E$39.2, E$4.2, PROGRAM.P$6
- new net S$23: E$1.24, E$22.2, E$27.1, E$37.C, E$8.TP
- new net S$24: E$1.21, E$24.TP, E$25.C, E$33.2, E$38.2
- net 5V: now also E$1.20, E$1.7, E$33.1, E$34.1, E$39.1, E$5.2; no longer E$1.21, E$25.C, E$33.2, E$38.2, E$8.1
- net S$13: no longer E$24.2
- net S$19: now also E$1.14, E$44.TP; no longer E$1.24, E$17.1, E$22.2, E$27.1, E$37.C
- net S$20: now also E$1.13, E$1.4; no longer E$1.22, E$1.8, E$12.2, E$15.1, E$19.1, E$2.P$7, E$24.1, E$29.2, E$3.1, E$3.2, E$3.3, E$3.4, E$3.5, E$34.2, E$36.2, E$38.1, E$39.2, E$5.2, PROGRAM.P$6
- net S$21: now also E$1.23, E$21.2, E$32.3; no longer E$1.20, E$1.7, E$34.1, E$39.1
- net S$7: now also E$17.3
- net S$8: now also E$9.TP
Routing:
- net S$18: track 0.00 -> 437.4 mm
- net S$7: track 0.00 -> 240.2 mm
- net 5V: track 0.00 -> 132.8 mm
- net S$23: track 0.00 -> 115.1 mm
- net S$13: track 0.00 -> 59.9 mm
- net S$20: track 0.00 -> 58.7 mm
- net S$12: track 0.00 -> 53.9 mm
- net S$11: track 0.00 -> 45.4 mm
- net S$10: track 0.00 -> 38.1 mm
- net S$21: track 0.00 -> 37.3 mm
- net S$14: track 0.00 -> 36.0 mm
- net S$24: track 0.00 -> 34.8 mm
- net S$15: track 0.00 -> 23.9 mm
- net S$16: track 0.00 -> 22.1 mm
- net S$3: track 0.00 -> 15.1 mm
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Other:
- board size 100.3 x 70 mm -> 100.3 x 69.8 mm

Commit message: .
Parts:
- added E$14: tx_to_multiplx, testpad:P1-17Y
Connections:
- net S$20: now also E$14.TP
Routing:
- net S$21: track 37.3 -> 55.6 mm
- net S$20: track 58.7 -> 62.1 mm
Changed lines of the file:
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@@
 <wire x1="1" y1="0" x2="101.33" y2="0" width="0.4064" layer="20"/>
 <wire x1="101.33" y1="0" x2="101.33" y2="69.85" width="0.4064" layer="20"/>
-<text x="80.138846875" y="1.536115625" size="1.27" layer="27">program</text>
-<text x="32.79225625" y="13.147590625" size="1.27" layer="27" rot="R180">debug</text>
+<text x="88.138846875" y="2.036115625" size="1.27" layer="27">program</text>
+<text x="34.29225625" y="3.647590625" size="1.27" layer="27" rot="R180">debug</text>
 <text x="34.925" y="16.51" size="1.27" layer="37" rot="R90">serial out</text>
 <text x="8.255" y="43.815" size="5.08" layer="21" rot="R90">-</text>
@@
 <rectangle x1="42.5" y1="15.5" x2="43" y2="17" layer="16"/>
 <rectangle x1="42.5" y1="15.5" x2="45.5" y2="22.5" layer="16"/>
-<rectangle x1="53" y1="19.5" x2="57.5" y2="23" layer="16"/>
 <rectangle x1="49" y1="8.5" x2="52.5" y2="11" layer="16"/>
 <rectangle x1="64" y1="11.5" x2="67.5" y2="14" layer="16"/>
@@
 <element name="E$7" library="eagle-ltspice" library_urn="urn:adsk.eagle:library:217" package="DIODE_F126Z12" package3d_urn="urn:adsk.eagle:package:13316/1" value="zener 60v" x="67.4" y="61" smashed="yes">
 <attribute name="NAME" x="64.225" y="62.778" size="1.27" layer="25" ratio="10"/>
-<attribute name="VALUE" x="63.655040625" y="57.251975" size="1.27" layer="27" ratio="10"/>
+<attribute name="VALUE" x="64.155040625" y="62.751975" size="1.27" layer="27" ratio="10"/>
 </element>
 <element name="E$10" library="crystal" library_urn="urn:adsk.eagle:library:204" package="HC49/S" package3d_urn="urn:adsk.eagle:package:12071/1" value="16Mhz" x="68.975" y="23.225" smashed="yes">
@@
 <element name="E$12" library="rcl" library_urn="urn:adsk.eagle:library:334" package="C025-024X044" package3d_urn="urn:adsk.eagle:package:23630/1" value="22p" x="61.09911875" y="22.844228125" smashed="yes" rot="R180">
 <attribute name="NAME" x="62.87711875" y="21.447228125" size="1.27" layer="25" ratio="10" rot="R180"/>
-<attribute name="VALUE" x="60.33711875" y="20.812228125" size="1.27" layer="27" ratio="10" rot="R270"/>
+<attribute name="VALUE" x="60.687771875" y="20.33711875" size="1.27" layer="27" ratio="10"/>
 </element>
 <element name="E$15" library="rcl" library_urn="urn:adsk.eagle:library:334" package="C025-024X044" package3d_urn="urn:adsk.eagle:package:23630/1" value="22p" x="77.225" y="23.405" smashed="yes" rot="R180">
 <attribute name="NAME" x="79.003" y="22.008" size="1.27" layer="25" ratio="10" rot="R180"/>
-<attribute name="VALUE" x="77.098" y="21.373" size="1.27" layer="27" ratio="10" rot="R270"/>
+<attribute name="VALUE" x="76.127" y="20.598" size="1.27" layer="27" ratio="10"/>
 </element>
 <element name="E$1" library="LSGPackages" package="ATMEGA328" value="" x="61.26" y="33.75" smashed="yes"/>
@@
 </element>
 <element name="E$37" library="diodes-zener" package="DO35-7" value="5v1 zener" x="81.4" y="53" smashed="yes" rot="R180">
-<attribute name="DIODEZENER" value="5v1-zener" x="84.4" y="51" size="1.27" layer="27" rot="R180"/>
+<attribute name="DIODEZENER" value="5v1-zener" x="86.4" y="51" size="1.27" layer="27" rot="R180"/>
 <attribute name="NAME" x="81.4" y="51.73" size="0.8128" layer="25" ratio="15" rot="R180" align="bottom-center"/>
 </element>
@@
 </element>
 <element name="E$25" library="diodes-zener" package="DO35-7" value="5v1 zener" x="68.2" y="54.2" smashed="yes">
-<attribute name="DIODEZENER" value="4v7-zener" x="65.2" y="56.2" size="1.27" layer="27"/>
+<attribute name="DIODEZENER" value="4v7-zener" x="65.2" y="55.7" size="1.27" layer="27"/>
 <attribute name="NAME" x="68.2" y="55.47" size="0.8128" layer="25" ratio="15" align="bottom-center"/>
 </element>
@@
 <element name="E$34" library="rcl" library_urn="urn:adsk.eagle:library:334" package="C025-024X044" package3d_urn="urn:adsk.eagle:package:23630/1" value="1uF" x="61" y="26" smashed="yes">
 <attribute name="NAME" x="59.222" y="27.397" size="1.27" layer="25" ratio="10"/>
-<attribute name="VALUE" x="56.968" y="26.127" size="1.27" layer="27" ratio="10" rot="R180"/>
+<attribute name="VALUE" x="58.468" y="27.127" size="1.27" layer="27" ratio="10" rot="R180"/>
 </element>
 <element name="E$38" library="rcl" library_urn="urn:adsk.eagle:library:334" package="C025-024X044" package3d_urn="urn:adsk.eagle:package:23630/1" value="0.1uF" x="63.2" y="44.8" smashed="yes">
@@
 <element name="E$44" library="testpad" library_urn="urn:adsk.eagle:library:385" package="P1-17Y" package3d_urn="urn:adsk.eagle:package:27953/1" value="tx_to_multiplx" x="82.84505625" y="30.47479375" smashed="yes" rot="R90">
 <attribute name="NAME" x="80.55905625" y="29.33179375" size="1.27" layer="25" ratio="10" rot="R90"/>
-<attribute name="TX_TO_MULTIPLX" value="tx_to_multiplx" x="85.56005625" y="34.18979375" size="1.016" layer="27" rot="R180"/>
+<attribute name="TX_TO_MULTIPLX" value="tx_to_multiplx" x="85.56005625" y="33.18979375" size="1.016" layer="27" rot="R180"/>
 <attribute name="VALUE" x="82.84505625" y="31.47479375" size="0.0254" layer="27" rot="R90"/>
 </element>
@@
 <attribute name="NAME" x="55.903796875" y="50.329346875" size="1.27" layer="25" ratio="10" rot="R90"/>
 <attribute name="VALUE" x="57.189796875" y="50.472346875" size="0.0254" layer="27" rot="R90"/>
-<attribute name="VOLTAGE_DIVIDER" value="aref" x="55.404796875" y="52.687346875" size="1.016" layer="27" rot="R180"/>
+<attribute name="VOLTAGE_DIVIDER" value="aref" x="62.904796875" y="50.687346875" size="1.016" layer="27" rot="R180"/>
 </element>
 <element name="E$41" library="solpad" library_urn="urn:adsk.eagle:library:364" package="LSP10" package3d_urn="urn:adsk.eagle:package:26501/1" value="" x="48.262375" y="48.9086625" smashed="yes">
@@
 <attribute name="NAME" x="75.644525" y="55.65643125" size="1.27" layer="25" ratio="10" rot="R90"/>
 <attribute name="VALUE" x="76.930525" y="55.79943125" size="0.0254" layer="27" rot="R90"/>
-<attribute name="VOLTAGE_DIVIDER" value="aref" x="75.145525" y="58.01443125" size="1.016" layer="27" rot="R180"/>
+<attribute name="VOLTAGE_DIVIDER" value="aref" x="75.645525" y="59.01443125" size="1.016" layer="27" rot="R180"/>
 </element>
 <element name="E$11" library="solpad" library_urn="urn:adsk.eagle:library:364" package="LSP10" package3d_urn="urn:adsk.eagle:package:26501/1" value="" x="90.04815" y="50.427065625" smashed="yes">
 <attribute name="NAME" x="88.77815" y="51.697065625" size="1.27" layer="25" ratio="10"/>
 <attribute name="VALUE" x="90.04815" y="50.681065625" size="0.0254" layer="27"/>
+</element>
+<element name="E$14" library="testpad" library_urn="urn:adsk.eagle:library:385" package="P1-17Y" package3d_urn="urn:adsk.eagle:package:27953/1" value="tx_to_multiplx" x="55.34505625" y="21.47479375" smashed="yes" rot="R90">
+<attribute name="INT0" value="int_in_attiny" x="59.56005625" y="20.18979375" size="1.016" layer="27" rot="R180"/>
+<attribute name="NAME" x="53.05905625" y="20.33179375" size="1.27" layer="25" ratio="10" rot="R90"/>
+<attribute name="VALUE" x="55.34505625" y="22.47479375" size="0.0254" layer="27" rot="R90"/>
 </element>
 </elements>
@@
 <wire x1="57.6" y1="39.99" x2="57.6" y2="42.431625" width="0.7" layer="16"/>
 <wire x1="44.428571875" y1="51.4" x2="44.45" y2="51.42" width="0.7" layer="16"/>
+<wire x1="57.6" y1="42.431625" x2="39.3" y2="42.431625" width="1.27" layer="16"/>
 </signal>
 <signal name="S$15">
@@
 <contactref element="E$1" pad="4"/>
 <wire x1="51" y1="18.1" x2="51" y2="27.34865" width="1.016" layer="16"/>
-<wire x1="81" y1="18.1" x2="51" y2="18.1" width="1.27" layer="16"/>
+<wire x1="51" y1="18.1" x2="55.5" y2="18.1" width="1.27" layer="16"/>
+<wire x1="55.5" y1="18.1" x2="81" y2="18.1" width="1.27" layer="16"/>
 <wire x1="81" y1="25.8" x2="81" y2="18.1" width="1.27" layer="16"/>
 <wire x1="77.38884375" y1="25.8" x2="81" y2="25.8" width="0.7" layer="16"/>
@@
 <wire x1="52.37" y1="28.9778375" x2="51" y2="27.34865" width="1.27" layer="16"/>
 <wire x1="75.240721875" y1="29.922528125" x2="75.23" y2="29.94" width="0.7" layer="16"/>
+<contactref element="E$14" pad="TP"/>
+<wire x1="55.34505625" y1="21.47479375" x2="55.34505625" y2="18.25494375" width="1.27" layer="16"/>
+<wire x1="55.34505625" y1="18.25494375" x2="55.5" y2="18.1" width="1.27" layer="16"/>
 </signal>
 <signal name="S$19">
