File: circuits/board/watts_meter.brd (EAGLE design)
At the start: 100.3 x 69.8 mm, 68 parts

Commit message: .
Parts:
- moved E$7 0.65 mm to (67.4, 61.7)
Connections:
- net S$18 renamed GROUND
Routing:
- net GROUND: track 437.4 -> 438.2 mm
Other:
- board size 100.3 x 69.8 mm -> 100 x 70 mm
Changed lines of the file:
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@@
 <setting verticaltext="up"/>
 </settings>
-<grid distance="0.5" unitdist="mm" unit="mm" style="lines" multiple="1" display="yes" altdistance="0.003125" altunitdist="mic" altunit="mm"/>
+<grid distance="1" unitdist="mm" unit="mm" style="lines" multiple="1" display="yes" altdistance="0.003125" altunitdist="mic" altunit="mm"/>
 <layers>
 <layer number="1" name="Top" color="4" fill="1" visible="yes" active="yes"/>
@@
 </layers>
 <board>
+<fusionsync huburn="a.cGVyc29uYWw6dWUyZDdmOThi" projecturn="a.cGVyc29uYWw6dWUyZDdmOThiIzIwMjAxMTA1MzUwMDc2Njgx" f3durn="urn:adsk.wipprod:dm.lineage:XYcBunLLQjmxC5qdX1j8Kw" pcbguid="2d6773c9-e221-43eb-a3cf-87bfbd118023" lastpulledtime="" lastsyncedchangeguid="21e963af-92a6-c428-d387-f30bb266baeb"/>
 <plain>
-<wire x1="1" y1="0" x2="1" y2="69.85" width="0.4064" layer="20"/>
-<wire x1="1" y1="69.85" x2="101" y2="69.85" width="0.4064" layer="20"/>
-<wire x1="1" y1="0" x2="101.33" y2="0" width="0.4064" layer="20"/>
-<wire x1="101.33" y1="0" x2="101.33" y2="69.85" width="0.4064" layer="20"/>
+<wire x1="1" y1="0" x2="1" y2="70" width="0.4064" layer="20"/>
+<wire x1="1" y1="0" x2="101" y2="0" width="0.4064" layer="20"/>
+<wire x1="101" y1="0" x2="101" y2="70" width="0.4064" layer="20"/>
 <text x="88.138846875" y="2.036115625" size="1.27" layer="27">program</text>
 <text x="34.29225625" y="3.647590625" size="1.27" layer="27" rot="R180">debug</text>
@@
 <rectangle x1="38.5" y1="54" x2="45.5" y2="63" layer="16"/>
 <rectangle x1="71" y1="5.5" x2="81" y2="7.5" layer="16"/>
-<rectangle x1="-19" y1="-6.5" x2="0.5" y2="87" layer="16"/>
-<rectangle x1="-19" y1="70.5" x2="119" y2="87" layer="16"/>
-<rectangle x1="-19" y1="-16.5" x2="125.5" y2="-0.5" layer="16"/>
-<rectangle x1="101.5" y1="-7.5" x2="127.5" y2="81" layer="16"/>
+<wire x1="1" y1="70" x2="101" y2="70" width="0.4064" layer="20"/>
 </plain>
 <attributes>
@@
 <element name="PROGRAM" library="LSGPackages" package="USB-MICRO-PCB" value="Program" x="91.185" y="6.985" smashed="yes"/>
 <element name="E$2" library="LSGPackages" package="USBMINIB" value="" x="31.48" y="11.43" smashed="yes" rot="R90"/>
-<element name="E$7" library="eagle-ltspice" library_urn="urn:adsk.eagle:library:217" package="DIODE_F126Z12" package3d_urn="urn:adsk.eagle:package:13316/1" value="zener 60v" x="67.4" y="61" smashed="yes">
-<attribute name="NAME" x="64.225" y="62.778" size="1.27" layer="25" ratio="10"/>
-<attribute name="VALUE" x="64.155040625" y="62.751975" size="1.27" layer="27" ratio="10"/>
+<element name="E$7" library="eagle-ltspice" library_urn="urn:adsk.eagle:library:217" package="DIODE_F126Z12" package3d_urn="urn:adsk.eagle:package:13316/1" value="zener 60v" x="67.4" y="61.650415625" smashed="yes">
+<attribute name="NAME" x="64.225" y="63.428415625" size="1.27" layer="25" ratio="10"/>
+<attribute name="VALUE" x="64.155040625" y="63.402390625" size="1.27" layer="27" ratio="10"/>
 </element>
 <element name="E$10" library="crystal" library_urn="urn:adsk.eagle:library:204" package="HC49/S" package3d_urn="urn:adsk.eagle:package:12071/1" value="16Mhz" x="68.975" y="23.225" smashed="yes">
@@
 <contactref element="E$13" pad="2"/>
 <contactref element="E$7" pad="C"/>
-<wire x1="60.55" y1="61.5" x2="61.05" y2="61" width="1.27" layer="16"/>
-<wire x1="60.55" y1="61.5" x2="53.8375" y2="61.5" width="1.27" layer="16"/>
+<wire x1="60.899584375" y1="61.5" x2="61.05" y2="61.650415625" width="1.27" layer="16"/>
+<wire x1="60.899584375" y1="61.5" x2="53.8375" y2="61.5" width="1.27" layer="16"/>
 </signal>
 <signal name="S$21">
@@
 <contactref element="E$20" pad="2"/>
 <contactref element="E$7" pad="A"/>
-<wire x1="73.75" y1="61" x2="78.5" y2="61" width="0.7" layer="16"/>
-<wire x1="78.5" y1="61" x2="78.59" y2="60.8" width="0.7" layer="16"/>
+<wire x1="73.75" y1="61.650415625" x2="78.2073125" y2="61.650415625" width="0.7" layer="16"/>
+<wire x1="78.2073125" y1="61.650415625" x2="78.59" y2="60.8" width="0.7" layer="16"/>
 <contactref element="E$9" pad="TP"/>
 <wire x1="77.59" y1="59.8" x2="77.59" y2="57.13995625" width="1.27" layer="16"/>
@@
 <wire x1="27.854346875" y1="35.34643125" x2="27.854346875" y2="35.911575" width="0.7" layer="16"/>
 </signal>
-<signal name="S$18">
+<signal name="GROUND">
 <contactref element="E$22" pad="3"/>
 <contactref element="E$3" pad="1"/>
@@
 <wire x1="61.5" y1="48.5" x2="61.5" y2="45.23" width="1.27" layer="16"/>
 <wire x1="61.93" y1="44.8" x2="61.5" y2="45.23" width="1.27" layer="16"/>
-<wire x1="41.8" y1="48.5" x2="44" y2="48.5" width="0.7" layer="16"/>
-<wire x1="41.8" y1="44.16151875" x2="41.8" y2="48.5" width="0.7" layer="16"/>
-<wire x1="61.16151875" y1="44.16151875" x2="41.8" y2="44.16151875" width="0.7" layer="16"/>
-<wire x1="44" y1="48.5" x2="44.45" y2="48.88" width="0.7" layer="16"/>
+<wire x1="41.518009375" y1="48.876028125" x2="44.445296875" y2="48.876028125" width="0.7" layer="16"/>
+<wire x1="41.518009375" y1="44.16151875" x2="41.518009375" y2="48.876028125" width="0.7" layer="16"/>
+<wire x1="61.16151875" y1="44.16151875" x2="41.518009375" y2="44.16151875" width="0.7" layer="16"/>
+<wire x1="44.445296875" y1="48.876028125" x2="44.45" y2="48.88" width="0.7" layer="16"/>
 <wire x1="91.5" y1="6" x2="86.5" y2="6" width="1.27" layer="16"/>
 <wire x1="95" y1="9.5" x2="91.5" y2="6" width="1.27" layer="16"/>
@@
 </note>
 <note version="8.3" severity="warning">
+Since Version 8.3, EAGLE supports Fusion synchronisation.
+This feature will not be available in this version and saving
+the document will break the link to the Fusion PCB feature.
+</note>
+<note version="8.3" severity="warning">
