File: circuits/board/watts_meter.brd (EAGLE design)
At the start: 100 x 70 mm, 68 parts

Commit message: rimosso errore su pin D7
Connections:
- new net S$4: E$1.13
- net S$20: no longer E$1.13
Routing:
- net S$20: track 62.1 -> 20.3 mm
Changed lines of the file:
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@@
 <wire x1="72.44444375" y1="40.44444375" x2="70.15" y2="37.56" width="1.016" layer="16"/>
 </signal>
+<signal name="S$4">
+<contactref element="E$1" pad="13"/>
+<wire x1="75.240721875" y1="29.922528125" x2="75.23" y2="29.94" width="0.7" layer="16"/>
+</signal>
 <signal name="S$20">
-<contactref element="E$1" pad="13"/>
 <contactref element="E$1" pad="4"/>
 <wire x1="51" y1="18.1" x2="51" y2="27.34865" width="1.016" layer="16"/>
-<wire x1="51" y1="18.1" x2="55.5" y2="18.1" width="1.27" layer="16"/>
-<wire x1="55.5" y1="18.1" x2="81" y2="18.1" width="1.27" layer="16"/>
-<wire x1="81" y1="25.8" x2="81" y2="18.1" width="1.27" layer="16"/>
-<wire x1="77.38884375" y1="25.8" x2="81" y2="25.8" width="0.7" layer="16"/>
-<wire x1="75.240721875" y1="27.948121875" x2="77.38884375" y2="25.8" width="0.7" layer="16"/>
-<wire x1="75.240721875" y1="29.922528125" x2="75.240721875" y2="27.948121875" width="0.7" layer="16"/>
+<wire x1="51" y1="18.1" x2="55.5" y2="18.1" width="1.016" layer="16"/>
 <wire x1="52.37" y1="28.9778375" x2="52.37" y2="29.94" width="0.7" layer="16"/>
 <wire x1="52.37" y1="28.9778375" x2="51" y2="27.34865" width="1.27" layer="16"/>
-<wire x1="75.240721875" y1="29.922528125" x2="75.23" y2="29.94" width="0.7" layer="16"/>
 <contactref element="E$14" pad="TP"/>
-<wire x1="55.34505625" y1="21.47479375" x2="55.34505625" y2="18.25494375" width="1.27" layer="16"/>
-<wire x1="55.34505625" y1="18.25494375" x2="55.5" y2="18.1" width="1.27" layer="16"/>
+<wire x1="55.5" y1="18.1" x2="55.5" y2="21.31985" width="1.016" layer="16"/>
+<wire x1="55.5" y1="21.31985" x2="55.34505625" y2="21.47479375" width="0.7" layer="16"/>
 </signal>
 <signal name="S$19">
